File: hardware/circuit/optional_i2c_device.kicad_sch (KiCad schematic)
At the start: 2 parts, among them U2 BMP581

Commit message: Release v0.19.0
Parts:
- U2: footprint inki:BMP581 -> Tinta:BMP581
Changed lines of the file:
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@@
 		)
 		(instances
-			(project "inki"
+			(project "tinta_l2"
 				(path "/240a819b-80d5-474c-958b-cef4297f8f8c/8aac0e89-39a1-4909-a5ea-b7760d4f132b"
 					(reference "C7")
@@
 			)
 		)
-		(property "Footprint" "inki:BMP581"
+		(property "Footprint" "Tinta:BMP581"
 			(at 77.47 41.91 0)
 			(effects
@@
 		)
 		(instances
-			(project "inki"
+			(project "tinta_l2"
 				(path "/240a819b-80d5-474c-958b-cef4297f8f8c/8aac0e89-39a1-4909-a5ea-b7760d4f132b"
 					(reference "U2")
