File: hardware/circuit/tinta_l2.kicad_pcb (KiCad board)
At the start: 2 copper layers, 47.2 x 55.5 mm, 60 parts, among them J1 connector epaper, J2 antenna, J3 Battery 3xAA/AAA, J6 pushbuttons, J7 status LED, Q1 2602, Q2 3904, Q3 2602, Q4 3904, U2 BMP581, U4 RV-3028, U5 ST25

Commit message: Release v0.19.0
Parts:
- U2: footprint inki:BMP581 -> Tinta:BMP581
Changed lines of the file:
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@@
 		(property ki_fp_filters "Connector*:*_1x??_*")
 		(sheetname "/")
-		(sheetfile "inki_l2.kicad_sch")
+		(sheetfile "tinta_l2.kicad_sch")
 		(attr through_hole)
 		(fp_line
@@
 		)
 		(sheetname "/")
-		(sheetfile "inki_l2.kicad_sch")
+		(sheetfile "tinta_l2.kicad_sch")
 		(attr smd)
 		(fp_line
@@
 		)
 		(sheetname "/")
-		(sheetfile "inki_l2.kicad_sch")
+		(sheetfile "tinta_l2.kicad_sch")
 		(attr smd)
 		(fp_line
@@
 		(property ki_fp_filters "Connector*:*_1x??_*")
 		(sheetname "/")
-		(sheetfile "inki_l2.kicad_sch")
+		(sheetfile "tinta_l2.kicad_sch")
 		(attr through_hole)
 		(fp_line
@@
 		(property ki_fp_filters "Connector*:*_1x??_*")
 		(sheetname "/")
-		(sheetfile "inki_l2.kicad_sch")
+		(sheetfile "tinta_l2.kicad_sch")
 		(attr through_hole)
 		(fp_line
@@
 		)
 	)
-	(footprint "inki:BMP581"
+	(footprint "Tinta:BMP581"
 		(layer "B.Cu")
 		(at 32.2 50.7375 180)
@@
 		)
 		(embedded_fonts no)
-		(model "${KICAD8_3DMODEL_DIR}/Package_LGA.3dshapes/Bosch_LGA-8_2x2.5mm_P0.65mm_ClockwisePinNumbering.wrl"
+		(model "${KICAD9_3DMODEL_DIR}/Package_LGA.3dshapes/Bosch_LGA-8_2x2.5mm_P0.65mm_ClockwisePinNumbering.step"
 			(offset
 				(xyz 0 0 0)
@@
 		(property ki_fp_filters "R_*")
 		(sheetname "/")
-		(sheetfile "inki_l2.kicad_sch")
+		(sheetfile "tinta_l2.kicad_sch")
 		(attr smd)
 		(fp_line
@@
 		(property ki_fp_filters "R_*")
 		(sheetname "/")
-		(sheetfile "inki_l2.kicad_sch")
+		(sheetfile "tinta_l2.kicad_sch")
 		(attr smd)
 		(fp_line
@@
 		(property ki_fp_filters "SOT?23*")
 		(sheetname "/")
-		(sheetfile "inki_l2.kicad_sch")
+		(sheetfile "tinta_l2.kicad_sch")
 		(attr smd)
 		(fp_line
@@
 		(property ki_fp_filters "R_*")
 		(sheetname "/")
-		(sheetfile "inki_l2.kicad_sch")
+		(sheetfile "tinta_l2.kicad_sch")
 		(attr smd)
 		(fp_line
@@
 		(property ki_fp_filters "SOT?23*")
 		(sheetname "/")
-		(sheetfile "inki_l2.kicad_sch")
+		(sheetfile "tinta_l2.kicad_sch")
 		(attr smd)
 		(fp_line
@@
 		(property ki_fp_filters "R_*")
 		(sheetname "/")
-		(sheetfile "inki_l2.kicad_sch")
+		(sheetfile "tinta_l2.kicad_sch")
 		(attr smd)
 		(fp_line
@@
 		(property ki_fp_filters "R_*")
 		(sheetname "/")
-		(sheetfile "inki_l2.kicad_sch")
+		(sheetfile "tinta_l2.kicad_sch")
 		(attr smd)
 		(fp_line
@@
 		(property ki_fp_filters "D*SOD?323F*")
 		(sheetname "/")
-		(sheetfile "inki_l2.kicad_sch")
+		(sheetfile "tinta_l2.kicad_sch")
 		(attr smd)
 		(fp_line
@@
 		)
 		(embedded_fonts no)
+		(model "${KICAD9_3DMODEL_DIR}/Package_SO.3dshapes/SOIC-8_3.9x4.9mm_P1.27mm.step"
+			(offset
+				(xyz 0 0 0)
+			)
+			(scale
+				(xyz 1 1 1)
+			)
+			(rotate
+				(xyz 0 0 0)
+			)
+		)
 	)
 	(footprint "Capacitor_SMD:C_0805_2012Metric"
@@
 		(property ki_fp_filters "R_*")
 		(sheetname "/")
-		(sheetfile "inki_l2.kicad_sch")
+		(sheetfile "tinta_l2.kicad_sch")
 		(attr smd)
 		(fp_line
@@
 		(property ki_fp_filters "R_*")
 		(sheetname "/")
-		(sheetfile "inki_l2.kicad_sch")
+		(sheetfile "tinta_l2.kicad_sch")
 		(attr smd)
 		(fp_line
@@
 		(property ki_fp_filters "R_*")
 		(sheetname "/")
-		(sheetfile "inki_l2.kicad_sch")
+		(sheetfile "tinta_l2.kicad_sch")
 		(attr smd)
 		(fp_line
@@
 		(property ki_fp_filters "R_*")
 		(sheetname "/")
-		(sheetfile "inki_l2.kicad_sch")
+		(sheetfile "tinta_l2.kicad_sch")
 		(attr smd)
 		(fp_line
@@
 		(property ki_fp_filters "C_*")
 		(sheetname "/")
-		(sheetfile "inki_l2.kicad_sch")
+		(sheetfile "tinta_l2.kicad_sch")
 		(attr smd)
 		(fp_line
@@
 		(property ki_fp_filters "D*SOD?323*")
 		(sheetname "/")
-		(sheetfile "inki_l2.kicad_sch")
+		(sheetfile "tinta_l2.kicad_sch")
 		(attr smd)
 		(fp_line
@@
 		(property ki_fp_filters "R_*")
 		(sheetname "/")
-		(sheetfile "inki_l2.kicad_sch")
+		(sheetfile "tinta_l2.kicad_sch")
 		(attr smd)
 		(fp_line
@@
 		(property ki_fp_filters "C_*")
 		(sheetname "/")
-		(sheetfile "inki_l2.kicad_sch")
+		(sheetfile "tinta_l2.kicad_sch")
 		(attr smd)
 		(fp_line
@@
 		(property ki_fp_filters "R_*")
 		(sheetname "/")
-		(sheetfile "inki_l2.kicad_sch")
+		(sheetfile "tinta_l2.kicad_sch")
 		(attr smd)
 		(fp_line
@@
 		(property ki_fp_filters "R_*")
 		(sheetname "/")
-		(sheetfile "inki_l2.kicad_sch")
+		(sheetfile "tinta_l2.kicad_sch")
 		(attr smd)
 		(fp_line
@@
 		(property ki_fp_filters "R_*")
 		(sheetname "/")
-		(sheetfile "inki_l2.kicad_sch")
+		(sheetfile "tinta_l2.kicad_sch")
 		(attr smd)
 		(fp_line
@@
 		(property ki_fp_filters "R_*")
 		(sheetname "/")
-		(sheetfile "inki_l2.kicad_sch")
+		(sheetfile "tinta_l2.kicad_sch")
 		(attr smd)
 		(fp_line
@@
 		(property ki_fp_filters "R_*")
 		(sheetname "/")
-		(sheetfile "inki_l2.kicad_sch")
+		(sheetfile "tinta_l2.kicad_sch")
 		(attr smd)
 		(fp_line
@@
 		(property ki_fp_filters "R_*")
 		(sheetname "/")
-		(sheetfile "inki_l2.kicad_sch")
+		(sheetfile "tinta_l2.kicad_sch")
 		(attr smd)
 		(fp_line
@@
 		(property ki_fp_filters "SOT?23*")
 		(sheetname "/")
-		(sheetfile "inki_l2.kicad_sch")
+		(sheetfile "tinta_l2.kicad_sch")
 		(attr smd)
 		(fp_line
@@
 		(property ki_fp_filters "SOT?23*")
 		(sheetname "/")
-		(sheetfile "inki_l2.kicad_sch")
+		(sheetfile "tinta_l2.kicad_sch")
 		(attr smd)
 		(fp_line
@@
 		(property ki_fp_filters "R_*")
 		(sheetname "/")
-		(sheetfile "inki_l2.kicad_sch")
+		(sheetfile "tinta_l2.kicad_sch")
 		(attr smd)
 		(fp_line
@@
 		(property ki_fp_filters "R_*")
 		(sheetname "/")
-		(sheetfile "inki_l2.kicad_sch")
+		(sheetfile "tinta_l2.kicad_sch")
 		(attr smd)
 		(fp_line
